File: can.kicad_sch (KiCad schematic)
At the start: 11 parts, among them U4 SN65HVD230

Commit message: New Template Update
Parts:
- C16: renamed from C34; footprint Capacitor_SMD:C_0603_1608Metric -> Capacitor_SMD:C_0402_1005Metric
- C19: renamed from C37; value 220 pF -> 220pF
- R8: renamed from R28; value 10k -> 0
- renumbered C33 to C15, C35 to C17, C36 to C18, D12 to D1, R30 to R10, R29 to R9, U4 to U2
Changed lines of the file:
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@@
   (symbol (lib_id "power:GND") (at 134.62 99.06 0) (unit 1)
     (in_bom yes) (on_board yes) (fields_autoplaced)
-    (property "Reference" "#PWR0130" (id 0) (at 134.62 105.41 0)
+    (property "Reference" "#PWR026" (id 0) (at 134.62 105.41 0)
       (effects (font (size 1.27 1.27)) hide)
     )
@@
   (symbol (lib_id "power:+3.3V") (at 124.46 68.58 0) (unit 1)
     (in_bom yes) (on_board yes) (fields_autoplaced)
-    (property "Reference" "#PWR0131" (id 0) (at 124.46 72.39 0)
+    (property "Reference" "#PWR024" (id 0) (at 124.46 72.39 0)
       (effects (font (size 1.27 1.27)) hide)
     )
@@
   (symbol (lib_id "Interface_CAN_LIN:SN65HVD230") (at 134.62 87.63 0) (unit 1)
     (in_bom yes) (on_board yes) (fields_autoplaced)
-    (property "Reference" "U4" (id 0) (at 142.24 75.1586 0))
+    (property "Reference" "U2" (id 0) (at 142.24 75.1586 0))
     (property "Value" "SN65HVD230" (id 1) (at 142.24 77.47 0))
     (property "Footprint" "Package_SO:SOIC-8_3.9x4.9mm_P1.27mm" (id 2) (at 134.62 100.33 0)
@@
   (symbol (lib_id "Device:C_Small") (at 127 71.12 0) (unit 1)
     (in_bom yes) (on_board yes) (fields_autoplaced)
-    (property "Reference" "C34" (id 0) (at 129.54 69.8562 0)
+    (property "Reference" "C16" (id 0) (at 129.54 69.8562 0)
       (effects (font (size 1.27 1.27)) (justify left))
     )
@@
       (effects (font (size 1.27 1.27)) (justify left))
     )
-    (property "Footprint" "Capacitor_SMD:C_0603_1608Metric" (id 2) (at 127 71.12 0)
+    (property "Footprint" "Capacitor_SMD:C_0402_1005Metric" (id 2) (at 127 71.12 0)
       (effects (font (size 1.27 1.27)) hide)
     )
@@
   (symbol (lib_id "Device:C_Small") (at 175.26 82.55 180) (unit 1)
     (in_bom yes) (on_board yes)
-    (property "Reference" "C36" (id 0) (at 173.99 74.93 0)
+    (property "Reference" "C18" (id 0) (at 173.99 74.93 0)
       (effects (font (size 1.27 1.27)) (justify right))
     )
@@
   (symbol (lib_id "Diode:SM712_SOT23") (at 186.69 88.9 270) (unit 1)
     (in_bom yes) (on_board yes) (fields_autoplaced)
-    (property "Reference" "D12" (id 0) (at 190.5 87.63 90)
+    (property "Reference" "D1" (id 0) (at 190.5 87.63 90)
       (effects (font (size 1.27 1.27)) (justify left))
     )
@@
   (symbol (lib_id "power:GND") (at 175.26 88.9 0) (unit 1)
     (in_bom yes) (on_board yes) (fields_autoplaced)
-    (property "Reference" "#PWR0146" (id 0) (at 175.26 95.25 0)
+    (property "Reference" "#PWR027" (id 0) (at 175.26 95.25 0)
       (effects (font (size 1.27 1.27)) hide)
     )
@@
   (symbol (lib_id "power:GND") (at 175.26 102.87 0) (unit 1)
     (in_bom yes) (on_board yes) (fields_autoplaced)
-    (property "Reference" "#PWR0151" (id 0) (at 175.26 109.22 0)
+    (property "Reference" "#PWR028" (id 0) (at 175.26 109.22 0)
       (effects (font (size 1.27 1.27)) hide)
     )
@@
   (symbol (lib_id "Device:C_Small") (at 121.92 71.12 0) (unit 1)
     (in_bom yes) (on_board yes) (fields_autoplaced)
-    (property "Reference" "C33" (id 0) (at 114.3 69.85 0)
+    (property "Reference" "C15" (id 0) (at 114.3 69.85 0)
       (effects (font (size 1.27 1.27)) (justify left))
     )
@@
   (symbol (lib_id "Device:R_Small") (at 124.46 95.25 0) (unit 1)
     (in_bom yes) (on_board yes)
-    (property "Reference" "R28" (id 0) (at 118.11 93.98 0)
-      (effects (font (size 1.27 1.27)) (justify left))
-    )
-    (property "Value" "10k" (id 1) (at 118.11 96.52 0)
+    (property "Reference" "R8" (id 0) (at 118.11 93.98 0)
+      (effects (font (size 1.27 1.27)) (justify left))
+    )
+    (property "Value" "0" (id 1) (at 118.11 96.52 0)
       (effects (font (size 1.27 1.27)) (justify left))
     )
@@
   (symbol (lib_id "Device:R") (at 167.64 93.98 0) (unit 1)
     (in_bom yes) (on_board yes) (fields_autoplaced)
-    (property "Reference" "R30" (id 0) (at 162.56 92.71 0)
+    (property "Reference" "R10" (id 0) (at 162.56 92.71 0)
       (effects (font (size 1.27 1.27)) (justify left))
     )
@@
   (symbol (lib_id "Device:R") (at 167.64 83.82 0) (unit 1)
     (in_bom yes) (on_board yes) (fields_autoplaced)
-    (property "Reference" "R29" (id 0) (at 162.56 82.55 0)
+    (property "Reference" "R9" (id 0) (at 162.56 82.55 0)
       (effects (font (size 1.27 1.27)) (justify left))
     )
@@
   (symbol (lib_id "Device:C") (at 171.45 88.9 90) (unit 1)
     (in_bom yes) (on_board yes) (fields_autoplaced)
-    (property "Reference" "C35" (id 0) (at 171.45 82.55 90))
+    (property "Reference" "C17" (id 0) (at 171.45 82.55 90))
     (property "Value" "0.1uF" (id 1) (at 171.45 85.09 90))
     (property "Footprint" "Capacitor_SMD:C_0402_1005Metric" (id 2) (at 175.26 87.9348 0)
@@
   (symbol (lib_id "power:GND") (at 124.46 73.66 0) (unit 1)
     (in_bom yes) (on_board yes) (fields_autoplaced)
-    (property "Reference" "#PWR0145" (id 0) (at 124.46 80.01 0)
+    (property "Reference" "#PWR025" (id 0) (at 124.46 80.01 0)
       (effects (font (size 1.27 1.27)) hide)
     )
@@
   (symbol (lib_id "Device:C_Small") (at 175.26 100.33 180) (unit 1)
     (in_bom yes) (on_board yes) (fields_autoplaced)
-    (property "Reference" "C37" (id 0) (at 177.8 100.33 0)
-      (effects (font (size 1.27 1.27)) (justify right))
-    )
-    (property "Value" "220 pF" (id 1) (at 177.8 102.87 0)
-      (effects (font (size 1.27 1.27)) (justify right))
-    )
+    (property "Reference" "C19" (id 0) (at 177.8 99.0535 0)
+      (effects (font (size 1.27 1.27)) (justify right))
+    )
+    (property "Value" "220pF" (id 1) (at 177.8 101.5935 0)
+      (effects (font (size 1.27 1.27)) (justify right))
+    )
