File: usb-uart.kicad_sch (KiCad schematic)
At the start: 16 parts, among them J3 USB_C_Receptacle_USB2.0, U6 SC4216H, U7 LTC4411

Commit message: New Template Update
Parts:
- removed C20, C25: 10uF, Capacitor_SMD:C_0603_1608Metric, symbol Device:C_Small
- removed C23: 4.7uF, Capacitor_SMD:C_0603_1608Metric, symbol Device:C_Small
- removed R24: 56k, Resistor_SMD:R_0402_1005Metric, symbol Device:R_Small
- removed R25: 10k, Resistor_SMD:R_0402_1005Metric, symbol Device:R_Small
- removed U6: SC4216H, iclr:SOIC127P599X175-9N, symbol iclr:RT9025-25GSP
- removed U7: LTC4411, Package_TO_SOT_SMD:SOT-23-5, symbol iclr:LTC4411
- USBLED1: footprint LED_SMD:LED_0603_1608Metric -> Resistor_SMD:R_0402_1005Metric
- renumbered D4 to D2, J3 to J2, R15 to R11, R16 to R12, R18 to R13, TP17 to TP1, TP18 to TP2, TP19 to TP3
Connections:
- no-connect marks 5 -> 2
