File: CommBoard.kicad_sch (KiCad schematic)
At the start: 44 parts, among them J1 RBUS, U1 ESP32-S3, U5 LTC4411, Y1 40MHz±10ppm

Commit message: New Template Update
Parts:
- removed C22: 4.7uF, Capacitor_SMD:C_0603_1608Metric, symbol Device:C_Small
- removed D1, D2: LED_Small, Resistor_SMD:R_0402_1005Metric, symbol Device:LED_Small
- removed R2, R3, R5: 470, Resistor_SMD:R_0402_1005Metric, symbol Device:R_Small
- removed U5: LTC4411, Package_TO_SOT_SMD:SOT-23-5, symbol iclr:LTC4411
- added D4, D6: LED_Small, Resistor_SMD:R_0402_1005Metric, symbol Device:LED_Small
- added R14, R15, R19, R20: 470, Resistor_SMD:R_0402_1005Metric, symbol Device:R_Small
- C12: value C -> 4.2pF; footprint Capacitor_SMD:C_0603_1608Metric -> Capacitor_SMD:C_0402_1005Metric
- C13, C14: footprint Capacitor_SMD:C_0603_1608Metric -> Capacitor_SMD:C_0402_1005Metric
- C3: renamed from C1; footprint Capacitor_SMD:C_0603_1608Metric -> Capacitor_SMD:C_0402_1005Metric
- L1, L2: footprint Inductor_SMD:L_0603_1608Metric -> Inductor_SMD:L_0402_1005Metric
- R5: renamed from R1; value 50 -> 47.5; footprint (none) -> Resistor_SMD:R_0402_1005Metric
- R6: value 470 -> 499
- renumbered C4 to C1, C5 to C4, C6 to C5, C7 to C6, C8 to C7, C3 to C8, R7 to R1, R11 to R2, R8 to R3, R14 to R4, R4 to R7
Connections:
- net GND: now also D4.1 (K), D6.1 (K)
- net R95_RX: now also R15.2
- net R95_TX: now also R14.2
- net R96_RX: now also R20.2; no longer R6.2
- net R96_TX: now also R19.2
- net TXD: now also R6.1; no longer U1.45 (MTDO/JTAG/GPIO40)
- net RBUS_uC_V: now reaches J1.3 (Pin_3)
- net at D3.2 (A): now also R14.1
- net at D5.2 (A): now also R19.1; no longer R6.1
- net at U1.49 (U0TXD/PROG/GPIO43): now also R6.2
- new net: D4.2 (A), R15.1
- new net: D6.2 (A), R20.1
- no-connect marks 4 -> 3
Other:
- added sheet Power (power.kicad_sch)
- note added: "Radio Status LEDs"
- moved on the sheet: R2, TXLED1

Commit message: New Routing
Connections:
- no-connect marks 3 -> 27
Changed lines of the file:
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@@
   (junction (at 69.85 135.89) (diameter 0) (color 0 0 0 0)
   )
+  (no_connect (at 69.85 118.11))
+  (no_connect (at 135.89 90.17))
+  (no_connect (at 69.85 92.71))
+  (no_connect (at 135.89 92.71))
+  (no_connect (at 135.89 77.47))
+  (no_connect (at 135.89 82.55))
+  (no_connect (at 69.85 97.79))
+  (no_connect (at 69.85 105.41))
+  (no_connect (at 135.89 80.01))
+  (no_connect (at 69.85 100.33))
+  (no_connect (at 135.89 85.09))
+  (no_connect (at 135.89 69.85))
+  (no_connect (at 69.85 72.39))
+  (no_connect (at 135.89 110.49))
   (no_connect (at 69.85 77.47))
+  (no_connect (at 69.85 102.87))
+  (no_connect (at 69.85 120.65))
+  (no_connect (at 135.89 130.81))
+  (no_connect (at 69.85 95.25))
+  (no_connect (at 69.85 90.17))
+  (no_connect (at 69.85 74.93))
   (no_connect (at 135.89 113.03))
+  (no_connect (at 135.89 87.63))
   (no_connect (at 135.89 123.19))
+  (no_connect (at 69.85 115.57))
+  (no_connect (at 135.89 128.27))
+  (no_connect (at 135.89 72.39))
   (wire (pts (xy 30.48 191.77) (xy 30.48 190.5))
     (stroke (width 0) (type default) (color 0 0 0 0))
